File: hardware/C-Comparator/schematics/Anpassung und Kombinierer/Widerstandsnetzwerk/Widerstandsnetzwerk.kicad_pcb (KiCad board)
At the start: 2 copper layers, 1 part, among them J1 Conn_Coaxial

Commit message: commit on mac
Parts:
- moved J1 39.1 mm to (102.0, 54.0)

Commit message: commit on Asteroids
Parts:
- moved J1 42.5 mm to (59.5, 53.5), turned to 90 degrees
Changed lines of the file:
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@@
 	(footprint "C-Comparator:CONN_73330-0030_MOL"
 		(layer "F.Cu")
-		(at 102 54)
+		(at 59.5 53.5 90)
 		(property "Reference" "J1"
-			(at -0.1016 0 0)
+			(at -0.1016 0 90)
 			(layer "F.SilkS")
 			(effects
@@
 		)
 		(property "Value" "Conn_Coaxial"
-			(at 10.3378 0 0)
+			(at 10.3378 0 90)
 			(layer "F.Fab")
 			(effects
@@
 		)
 		(property "Datasheet" ""
-			(at 0 0 0)
+			(at 0 0 90)
 			(layer "F.Fab")
 			(hide yes)
@@
 		)
 		(property "Description" "coaxial connector (BNC, SMA, SMB, SMC, Cinch/RCA, LEMO, ...)"
-			(at 0 0 0)
+			(at 0 0 90)
 			(layer "F.Fab")
 			(hide yes)
@@
 		(duplicate_pad_numbers_are_jumpers no)
 		(fp_line
+			(start 4.8768 -23.5712)
+			(end -4.8768 -23.5712)
+			(stroke
+				(width 0.1524)
+				(type solid)
+			)
+			(layer "F.SilkS")
+		)
+		(fp_line
 			(start -4.8768 -23.5712)
 			(end -4.8768 -6.0706)
@@
 		)
 		(fp_line
+			(start 4.8768 -6.0706)
+			(end 4.8768 -23.5712)
+			(stroke
+				(width 0.1524)
+				(type solid)
+			)
+			(layer "F.SilkS")
+		)
+		(fp_line
+			(start 2.54 -4.8768)
+			(end -2.54 -4.8768)
+			(stroke
+				(width 0.1524)
+				(type solid)
+			)
+			(layer "F.SilkS")
+		)
+		(fp_line
+			(start -2.4638 -4.6228)
+			(end 2.4638 -4.6228)
+			(stroke
+				(width 0.1524)
+				(type solid)
+			)
+			(layer "F.SilkS")
+		)
+		(fp_line
 			(start -4.8768 -2.54)
 			(end -4.8768 2.54)
@@
 		)
 		(fp_line
+			(start 4.8768 2.54)
+			(end 4.8768 -2.54)
+			(stroke
+				(width 0.1524)
+				(type solid)
+			)
+			(layer "F.SilkS")
+		)
+		(fp_line
 			(start -2.54 4.8768)
 			(end 2.54 4.8768)
@@
 		)
 		(fp_line
-			(start -2.4638 -4.6228)
-			(end 2.4638 -4.6228)
-			(stroke
-				(width 0.1524)
-				(type solid)
-			)
-			(layer "F.SilkS")
-		)
-		(fp_line
-			(start 2.54 -4.8768)
-			(end -2.54 -4.8768)
-			(stroke
-				(width 0.1524)
-				(type solid)
-			)
-			(layer "F.SilkS")
-		)
-		(fp_line
-			(start 4.8768 -23.5712)
-			(end -4.8768 -23.5712)
-			(stroke
-				(width 0.1524)
-				(type solid)
-			)
-			(layer "F.SilkS")
-		)
-		(fp_line
-			(start 4.8768 -6.0706)
-			(end 4.8768 -23.5712)
-			(stroke
-				(width 0.1524)
-				(type solid)
-			)
-			(layer "F.SilkS")
-		)
-		(fp_line
-			(start 4.8768 2.54)
-			(end 4.8768 -2.54)
-			(stroke
-				(width 0.1524)
-				(type solid)
-			)
-			(layer "F.SilkS")
+			(start 4.7498 -23.4442)
+			(end -4.7498 -23.4442)
+			(stroke
+				(width 0.1524)
+				(type solid)
+			)
+			(layer "F.Fab")
 		)
 		(fp_line
@@
 		)
 		(fp_line
+			(start 4.7498 -4.7498)
+			(end 4.7498 -23.4442)
+			(stroke
+				(width 0.1524)
+				(type solid)
+			)
+			(layer "F.Fab")
+		)
+		(fp_line
+			(start 4.7498 -4.7498)
+			(end -4.7498 -4.7498)
+			(stroke
+				(width 0.1524)
+				(type solid)
+			)
+			(layer "F.Fab")
+		)
+		(fp_line
 			(start -4.7498 -4.7498)
 			(end -4.7498 4.7498)
@@
 		)
 		(fp_line
+			(start 4.7498 4.7498)
+			(end 4.7498 -4.7498)
+			(stroke
+				(width 0.1524)
+				(type solid)
+			)
+			(layer "F.Fab")
+		)
+		(fp_line
 			(start -4.7498 4.7498)
 			(end 4.7498 4.7498)
@@
 			(layer "F.Fab")
 		)
-		(fp_line
-			(start 4.7498 -23.4442)
-			(end -4.7498 -23.4442)
-			(stroke
-				(width 0.1524)
-				(type solid)
-			)
-			(layer "F.Fab")
-		)
-		(fp_line
-			(start 4.7498 -4.7498)
-			(end -4.7498 -4.7498)
-			(stroke
-				(width 0.1524)
-				(type solid)
-			)
-			(layer "F.Fab")
-		)
-		(fp_line
-			(start 4.7498 -4.7498)
-			(end 4.7498 -23.4442)
-			(stroke
-				(width 0.1524)
-				(type solid)
-			)
-			(layer "F.Fab")
-		)
-		(fp_line
-			(start 4.7498 4.7498)
-			(end 4.7498 -4.7498)
-			(stroke
-				(width 0.1524)
-				(type solid)
-			)
-			(layer "F.Fab")
-		)
 		(pad "1" thru_hole circle
-			(at 0 0)
+			(at 0 0 90)
 			(size 1.7526 1.7526)
 			(drill 1.2446)
@@
 		)
 		(pad "2" thru_hole circle
-			(at -4.318 -4.318)
+			(at -4.318 -4.318 90)
 			(size 3.048 3.048)
 			(drill 2.54)
@@
 		)
 		(pad "3" thru_hole circle
-			(at -4.318 4.318)
+			(at -4.318 4.318 90)
 			(size 3.048 3.048)
 			(drill 2.54)
@@
 		)
 		(pad "4" thru_hole circle
-			(at 4.318 4.318)
+			(at 4.318 4.318 90)
 			(size 3.048 3.048)
 			(drill 2.54)
@@
 		)
 		(pad "5" thru_hole circle
-			(at 4.318 -4.318)
-			(size 3.048 3.048)
-			(drill 2.54)
+			(at 4.318 -4.318 90)
+			(size 3.048 3.048)
+			(drill 2.54)

Commit message: commit on mac
Parts:
- moved J1 42.5 mm to (102.0, 54.0), turned to 0 degrees
Changed lines of the file:
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@@
 	(footprint "C-Comparator:CONN_73330-0030_MOL"
 		(layer "F.Cu")
-		(at 59.5 53.5 90)
+		(at 102 54)
 		(property "Reference" "J1"
-			(at -0.1016 0 90)
+			(at -0.1016 0 0)
 			(layer "F.SilkS")
 			(effects
@@
 		)
 		(property "Value" "Conn_Coaxial"
-			(at 10.3378 0 90)
+			(at 10.3378 0 0)
 			(layer "F.Fab")
 			(effects
@@
 		)
 		(property "Datasheet" ""
-			(at 0 0 90)
+			(at 0 0 0)
 			(layer "F.Fab")
 			(hide yes)
@@
 		)
 		(property "Description" "coaxial connector (BNC, SMA, SMB, SMC, Cinch/RCA, LEMO, ...)"
-			(at 0 0 90)
+			(at 0 0 0)
 			(layer "F.Fab")
 			(hide yes)
@@
 		(duplicate_pad_numbers_are_jumpers no)
 		(fp_line
+			(start -4.8768 -23.5712)
+			(end -4.8768 -6.0706)
+			(stroke
+				(width 0.1524)
+				(type solid)
+			)
+			(layer "F.SilkS")
+		)
+		(fp_line
+			(start -4.8768 -2.54)
+			(end -4.8768 2.54)
+			(stroke
+				(width 0.1524)
+				(type solid)
+			)
+			(layer "F.SilkS")
+		)
+		(fp_line
+			(start -2.54 4.8768)
+			(end 2.54 4.8768)
+			(stroke
+				(width 0.1524)
+				(type solid)
+			)
+			(layer "F.SilkS")
+		)
+		(fp_line
+			(start -2.4638 -4.6228)
+			(end 2.4638 -4.6228)
+			(stroke
+				(width 0.1524)
+				(type solid)
+			)
+			(layer "F.SilkS")
+		)
+		(fp_line
+			(start 2.54 -4.8768)
+			(end -2.54 -4.8768)
+			(stroke
+				(width 0.1524)
+				(type solid)
+			)
+			(layer "F.SilkS")
+		)
+		(fp_line
 			(start 4.8768 -23.5712)
 			(end -4.8768 -23.5712)
@@
 		)
 		(fp_line
-			(start -4.8768 -23.5712)
-			(end -4.8768 -6.0706)
-			(stroke
-				(width 0.1524)
-				(type solid)
-			)
-			(layer "F.SilkS")
-		)
-		(fp_line
 			(start 4.8768 -6.0706)
 			(end 4.8768 -23.5712)
@@
 		)
 		(fp_line
-			(start 2.54 -4.8768)
-			(end -2.54 -4.8768)
-			(stroke
-				(width 0.1524)
-				(type solid)
-			)
-			(layer "F.SilkS")
-		)
-		(fp_line
-			(start -2.4638 -4.6228)
-			(end 2.4638 -4.6228)
-			(stroke
-				(width 0.1524)
-				(type solid)
-			)
-			(layer "F.SilkS")
-		)
-		(fp_line
-			(start -4.8768 -2.54)
-			(end -4.8768 2.54)
-			(stroke
-				(width 0.1524)
-				(type solid)
-			)
-			(layer "F.SilkS")
-		)
-		(fp_line
 			(start 4.8768 2.54)
 			(end 4.8768 -2.54)
@@
 		)
 		(fp_line
-			(start -2.54 4.8768)
-			(end 2.54 4.8768)
-			(stroke
-				(width 0.1524)
-				(type solid)
-			)
-			(layer "F.SilkS")
+			(start -4.7498 -23.4442)
+			(end -4.7498 -4.7498)
+			(stroke
+				(width 0.1524)
+				(type solid)
+			)
+			(layer "F.Fab")
+		)
+		(fp_line
+			(start -4.7498 -4.7498)
+			(end -4.7498 4.7498)
+			(stroke
+				(width 0.1524)
+				(type solid)
+			)
+			(layer "F.Fab")
+		)
+		(fp_line
+			(start -4.7498 4.7498)
+			(end 4.7498 4.7498)
+			(stroke
+				(width 0.1524)
+				(type solid)
+			)
+			(layer "F.Fab")
 		)
 		(fp_line
@@
 		)
 		(fp_line
-			(start -4.7498 -23.4442)
+			(start 4.7498 -4.7498)
 			(end -4.7498 -4.7498)
 			(stroke
@@
 		)
 		(fp_line
-			(start 4.7498 -4.7498)
-			(end -4.7498 -4.7498)
-			(stroke
-				(width 0.1524)
-				(type solid)
-			)
-			(layer "F.Fab")
-		)
-		(fp_line
-			(start -4.7498 -4.7498)
-			(end -4.7498 4.7498)
-			(stroke
-				(width 0.1524)
-				(type solid)
-			)
-			(layer "F.Fab")
-		)
-		(fp_line
 			(start 4.7498 4.7498)
 			(end 4.7498 -4.7498)
@@
 			(layer "F.Fab")
 		)
-		(fp_line
-			(start -4.7498 4.7498)
-			(end 4.7498 4.7498)
-			(stroke
-				(width 0.1524)
-				(type solid)
-			)
-			(layer "F.Fab")
-		)
 		(pad "1" thru_hole circle
-			(at 0 0 90)
+			(at 0 0)
 			(size 1.7526 1.7526)
 			(drill 1.2446)
@@
 		)
 		(pad "2" thru_hole circle
-			(at -4.318 -4.318 90)
+			(at -4.318 -4.318)
 			(size 3.048 3.048)
 			(drill 2.54)
@@
 		)
 		(pad "3" thru_hole circle
-			(at -4.318 4.318 90)
+			(at -4.318 4.318)
 			(size 3.048 3.048)
 			(drill 2.54)
@@
 		)
 		(pad "4" thru_hole circle
-			(at 4.318 4.318 90)
+			(at 4.318 4.318)
 			(size 3.048 3.048)
 			(drill 2.54)
@@
 		)
 		(pad "5" thru_hole circle
-			(at 4.318 -4.318 90)
-			(size 3.048 3.048)
-			(drill 2.54)
+			(at 4.318 -4.318)
+			(size 3.048 3.048)
+			(drill 2.54)

Commit message: commit on Asteroids
Parts:
- moved J1 26.0 mm to (76.0, 53.5), turned to 90 degrees
Changed lines of the file:
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@@
 	(footprint "C-Comparator:CONN_73330-0030_MOL"
 		(layer "F.Cu")
-		(at 102 54)
+		(at 76 53.5 90)
 		(property "Reference" "J1"
-			(at -0.1016 0 0)
+			(at -0.1016 0 90)
 			(layer "F.SilkS")
 			(effects
@@
 		)
 		(property "Value" "Conn_Coaxial"
-			(at 10.3378 0 0)
+			(at 10.3378 0 90)
 			(layer "F.Fab")
 			(effects
@@
 		)
 		(property "Datasheet" ""
-			(at 0 0 0)
+			(at 0 0 90)
 			(layer "F.Fab")
 			(hide yes)
@@
 		)
 		(property "Description" "coaxial connector (BNC, SMA, SMB, SMC, Cinch/RCA, LEMO, ...)"
-			(at 0 0 0)
+			(at 0 0 90)
 			(layer "F.Fab")
 			(hide yes)
@@
 		(duplicate_pad_numbers_are_jumpers no)
 		(fp_line
+			(start 4.8768 -23.5712)
+			(end -4.8768 -23.5712)
+			(stroke
+				(width 0.1524)
+				(type solid)
+			)
+			(layer "F.SilkS")
+		)
+		(fp_line
 			(start -4.8768 -23.5712)
 			(end -4.8768 -6.0706)
@@
 		)
 		(fp_line
+			(start 4.8768 -6.0706)
+			(end 4.8768 -23.5712)
+			(stroke
+				(width 0.1524)
+				(type solid)
+			)
+			(layer "F.SilkS")
+		)
+		(fp_line
+			(start 2.54 -4.8768)
+			(end -2.54 -4.8768)
+			(stroke
+				(width 0.1524)
+				(type solid)
+			)
+			(layer "F.SilkS")
+		)
+		(fp_line
+			(start -2.4638 -4.6228)
+			(end 2.4638 -4.6228)
+			(stroke
+				(width 0.1524)
+				(type solid)
+			)
+			(layer "F.SilkS")
+		)
+		(fp_line
 			(start -4.8768 -2.54)
 			(end -4.8768 2.54)
@@
 		)
 		(fp_line
+			(start 4.8768 2.54)
+			(end 4.8768 -2.54)
+			(stroke
+				(width 0.1524)
+				(type solid)
+			)
+			(layer "F.SilkS")
+		)
+		(fp_line
 			(start -2.54 4.8768)
 			(end 2.54 4.8768)
@@
 		)
 		(fp_line
-			(start -2.4638 -4.6228)
-			(end 2.4638 -4.6228)
-			(stroke
-				(width 0.1524)
-				(type solid)
-			)
-			(layer "F.SilkS")
-		)
-		(fp_line
-			(start 2.54 -4.8768)
-			(end -2.54 -4.8768)
-			(stroke
-				(width 0.1524)
-				(type solid)
-			)
-			(layer "F.SilkS")
-		)
-		(fp_line
-			(start 4.8768 -23.5712)
-			(end -4.8768 -23.5712)
-			(stroke
-				(width 0.1524)
-				(type solid)
-			)
-			(layer "F.SilkS")
-		)
-		(fp_line
-			(start 4.8768 -6.0706)
-			(end 4.8768 -23.5712)
-			(stroke
-				(width 0.1524)
-				(type solid)
-			)
-			(layer "F.SilkS")
-		)
-		(fp_line
-			(start 4.8768 2.54)
-			(end 4.8768 -2.54)
-			(stroke
-				(width 0.1524)
-				(type solid)
-			)
-			(layer "F.SilkS")
+			(start 4.7498 -23.4442)
+			(end -4.7498 -23.4442)
+			(stroke
+				(width 0.1524)
+				(type solid)
+			)
+			(layer "F.Fab")
 		)
 		(fp_line
@@
 		)
 		(fp_line
+			(start 4.7498 -4.7498)
+			(end 4.7498 -23.4442)
+			(stroke
+				(width 0.1524)
+				(type solid)
+			)
+			(layer "F.Fab")
+		)
+		(fp_line
+			(start 4.7498 -4.7498)
+			(end -4.7498 -4.7498)
+			(stroke
+				(width 0.1524)
+				(type solid)
+			)
+			(layer "F.Fab")
+		)
+		(fp_line
 			(start -4.7498 -4.7498)
 			(end -4.7498 4.7498)
@@
 		)
 		(fp_line
+			(start 4.7498 4.7498)
+			(end 4.7498 -4.7498)
+			(stroke
+				(width 0.1524)
+				(type solid)
+			)
+			(layer "F.Fab")
+		)
+		(fp_line
 			(start -4.7498 4.7498)
 			(end 4.7498 4.7498)
@@
 			(layer "F.Fab")
 		)
-		(fp_line
-			(start 4.7498 -23.4442)
-			(end -4.7498 -23.4442)
-			(stroke
-				(width 0.1524)
-				(type solid)
-			)
-			(layer "F.Fab")
-		)
-		(fp_line
-			(start 4.7498 -4.7498)
-			(end -4.7498 -4.7498)
-			(stroke
-				(width 0.1524)
-				(type solid)
-			)
-			(layer "F.Fab")
-		)
-		(fp_line
-			(start 4.7498 -4.7498)
-			(end 4.7498 -23.4442)
-			(stroke
-				(width 0.1524)
-				(type solid)
-			)
-			(layer "F.Fab")
-		)
-		(fp_line
-			(start 4.7498 4.7498)
-			(end 4.7498 -4.7498)
-			(stroke
-				(width 0.1524)
-				(type solid)
-			)
-			(layer "F.Fab")
-		)
 		(pad "1" thru_hole circle
-			(at 0 0)
+			(at 0 0 90)
 			(size 1.7526 1.7526)
 			(drill 1.2446)
@@
 		)
 		(pad "2" thru_hole circle
-			(at -4.318 -4.318)
+			(at -4.318 -4.318 90)
 			(size 3.048 3.048)
 			(drill 2.54)
@@
 		)
 		(pad "3" thru_hole circle
-			(at -4.318 4.318)
+			(at -4.318 4.318 90)
 			(size 3.048 3.048)
 			(drill 2.54)
@@
 		)
 		(pad "4" thru_hole circle
-			(at 4.318 4.318)
+			(at 4.318 4.318 90)
 			(size 3.048 3.048)
 			(drill 2.54)
@@
 		)
 		(pad "5" thru_hole circle
-			(at 4.318 -4.318)
-			(size 3.048 3.048)
-			(drill 2.54)
+			(at 4.318 -4.318 90)
+			(size 3.048 3.048)
+			(drill 2.54)

Commit message: commit on mac
Parts:
- moved J1 27.0 mm to (56.4, 72.0)
Changed lines of the file:
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@@
 	(footprint "C-Comparator:CONN_73330-0030_MOL"
 		(layer "F.Cu")
-		(at 76 53.5 90)
+		(at 56.4027 72 90)
 		(property "Reference" "J1"
 			(at -0.1016 0 90)

Commit message: PCB title
Other:
- board text added: "1.0"
- board text added: "2026-10-28"
- board text added: "Anpassung und Kombinierer für GPSDO+AWG/SDR auf Sat-Kabel"
Changed lines of the file:
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@@
 		(embedded_fonts no)
+	)
+	(gr_text "Anpassung und Kombinierer für GPSDO+AWG/SDR auf Sat-Kabel"
+		(at 187.5 190.5 0)
+		(layer "F.Cu")
+		(effects
+			(font
+				(size 1.5 1.5)
+				(thickness 0.3)
+				(bold yes)
+			)
+			(justify left bottom)
+		)
+	)
+	(gr_text "2026-10-28"
+		(at 206.5 194 0)
+		(layer "F.Cu")
+		(effects
+			(font
+				(size 1.5 1.5)
+				(thickness 0.3)
+				(bold yes)
+			)
+			(justify left bottom)
+		)
+	)
+	(gr_text "1.0"
+		(at 269 194 0)
+		(layer "F.Cu")
+		(effects
+			(font
+				(size 1.5 1.5)
+				(thickness 0.3)
+				(bold yes)
+			)
+			(justify left bottom)
+		)
 	)
 	(embedded_fonts no)

Commit message: Anpassung
Parts:
- added J3: AWG, Connector_Coaxial:SMA_Amphenol_132291_Vertical, F.Cu at (250.5, 151.0)
- added R1: 43,4 Ω, Resistor_THT:R_Axial_DIN0309_L9.0mm_D3.2mm_P12.70mm_Horizontal, F.Cu at (248.0, 81.2)
- added R2: 86,6 Ω, Resistor_THT:R_Axial_DIN0309_L9.0mm_D3.2mm_P12.70mm_Horizontal, F.Cu at (248.5, 111.2)
- J1: value Conn_Coaxial -> SATA IN
- moved J1 191.4 mm to (247.7, 65.3), turned to 0 degrees
Connections:
- J1 pad 1: unconnected-(J1-In-Pad1) -> Net-(J1-In)
- J1 pad 2: unconnected-(J1-Ext-Pad2) -> GND
