File: hardware/C-Comparator/schematics/Anpassung und Kombinierer/Widerstandsnetzwerk/Widerstandsnetzwerk.kicad_sch (KiCad schematic)
At the start: 2 parts, among them J1 SATA IN, J2 SATA OUT

Commit message: commit on mac
Other:
- moved on the sheet: J1

Commit message: Anpassung
Parts:
- added J3: AWG, Connector_Coaxial:SMA_Amphenol_132291_Vertical, symbol Connector_Generic_Shielded:Conn_01x01_Shielded
- added R1: 43,4 Ω, Resistor_THT:R_Axial_DIN0309_L9.0mm_D3.2mm_P12.70mm_Horizontal, symbol Device:R
- added R2: 86,6 Ω, Resistor_THT:R_Axial_DIN0309_L9.0mm_D3.2mm_P12.70mm_Horizontal, symbol Device:R
Connections:
- net at J1.1 (In): now also R1.1
- net GND: now reaches J1.2 (Ext)
- net GND: now also J3.SH (Shield), R2.2
- new net: J3.1 (Pin_1), R1.2, R2.1
